File: pico-dram-tester.kicad_pcb (KiCad board)
At the start: 2 copper layers, 100 x 100 mm, 44 parts, among them J1 TFT 4383, J2 mrd_114_ips_lcd_8p, Q1 XP9561GI, SW1 RotaryEncoder_Switch, SW2 BACK, U1 PICO2, U2 4116, U3 4132, U4 4164/41128/41256, U5 4416/4464, U6 44256, U7 DCDC_ITR03, U8 RFM-0505S, U9 APX803S

Commit message: Version 3 release
Parts:
- removed TP6: GND, TestPoint:TestPoint_Keystone_5005-5009_Compact
- added J3: POWER, Connector_USB:USB_C_Receptacle_GCT_USB4125-xx-x-0190_6P_TopMnt_Horizontal, F.Cu at (146.7, 53.4)
- added JP1: TYPE, Jumper:SolderJumper-2_P1.3mm_Open_Pad1.0x1.5mm, B.Cu at (125.7, 144.3)
- added R11: 5.1K, Passive:RESA500, F.Cu at (144.3, 59.6)
- added R12: 5.1K, Passive:RESA500, F.Cu at (144.3, 63.1)
- Q1: value XP9561GI -> SUP53P06-20-E3 or equiv
- R1, RN1, RN2, RN3, RN4: value 100 -> 33
- SW1: footprint Switch:PANASONIC_EVEY -> Switch:ENCODER_SW_UNIV
- U1: footprint Active:Pico2 -> Active:Pico2_PTH
- moved C1 20.7 mm to (159.6, 64.4), turned to -90 degrees
- moved TP4 4.06 mm to (137.2, 53.3)
- moved TP1 3.17 mm to (155.6, 53.3)
- moved TP3 2.67 mm to (160.7, 53.3)
- moved R4 1.14 mm to (144.3, 66.7)
- moved R5 1.14 mm to (144.3, 70.2)
- moved Q1 0.06 mm to (155.2, 68.7)
Routing:
- net VCC: track 147.5 -> 164.7 mm, vias 1 -> 3
- net Net-(J3-CC2): track 0.00 -> 8.46 mm
- net Net-(J3-CC1): track 0.00 -> 5.61 mm
- net /SP4: track 241.9 -> 246.8 mm
- net Net-(JP1-B): track 0.00 -> 3.94 mm
- net +12V: track 133.4 -> 137.3 mm
- net /SP3: track 219.5 -> 223.4 mm
- net /SP0: track 196.9 -> 200.0 mm
- net /SP8: track 115.2 -> 117.7 mm
- net /SP16: track 128.9 -> 126.6 mm
- net /SP9: track 174.8 -> 177.2 mm
- net Net-(RN3A-R1.2): track 53.0 -> 55.2 mm
- net /SP5: track 207.0 -> 209.1 mm
- net -5V: track 106.9 -> 108.6 mm
- net Net-(RN4B-R2.2): track 5.24 -> 6.86 mm
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Other:
- board text added: "Rev 3 6/26"
- board text added: "SHORT=BOURNS OPEN=PANASONIC"
- board text added: "© 2026 Tube Time"
- board text removed: "Rev 2 11/24"
- board text removed: "© 2024 Tube Time"
