File: pico-dram-tester.kicad_sch (KiCad schematic)
At the start: 44 parts, among them J1 TFT 4383, J2 mrd_114_ips_lcd_8p, Q1 SUP53P06-20-E3 or equiv, SW1 RotaryEncoder_Switch, SW2 BACK, U1 PICO2, U2 4116, U3 4132, U4 4164/41128/41256, U5 4416/4464, U6 44256, U7 DCDC_ITR03, U8 RFM-0505S, U9 APX803S

Commit message: Version 3 release
Parts:
- removed SW1: RotaryEncoder_Switch, Switch:PANASONIC_EVEY, symbol switches_new:RotaryEncoder_Sw_Panasonic_EVE
- removed TP6: GND, TestPoint:TestPoint_Keystone_5005-5009_Compact, symbol Connector:TestPoint
- added J3: POWER, Connector_USB:USB_C_Receptacle_GCT_USB4125-xx-x-0190_6P_TopMnt_Horizontal, symbol Connector:USB_C_Receptacle_PowerOnly_6P
- added JP1: TYPE, Jumper:SolderJumper-2_P1.3mm_Open_Pad1.0x1.5mm, symbol Jumper:Jumper_2_Small_Open
- added R11, R12: 5.1K, Passive:RESA500, symbol Device:R
- added SW1: RotaryEncoder_Switch, Switch:ENCODER_SW_UNIV, symbol switches_new:RotaryEncoder_Sw_Universal
- U1: footprint Active:Pico2 -> Active:Pico2_PTH
Connections:
- net GND: now also J3.A12 (GND), J3.B12 (GND), J3.S1 (SHIELD), JP1.1 (A), R11.2, R12.2, SW1.C, SW1.SH
- net VCC: now also J3.A9 (VBUS), J3.B9 (VBUS)
- net at R8.2, U1.29 (GP22): now also SW1.A
- net at R6.2, U1.32 (GP27/ADC1/I2C1_SCL): now also SW1.S
- net at R7.2, U1.31 (GP26/ADC0/I2C1_SDA): now also SW1.B
- new net: JP1.2 (B), SW1.C2 (C)
- new net: J3.A5 (CC1), R11.1
- new net: J3.B5 (CC2), R12.1
Other:
- note added: "(C) 2026 Tube Time"
- note added: "JP1: OPEN FOR PANASONIC SHORTED FOR BOURNS"
- note removed: "(C) 2024 Tube Time"
